File: HW/ESP-VINDRIKTNING_no_batt.brd (EAGLE design)
At the start: 30 x 75.6 mm, 47 parts, among them IC1 PI4ULS5V202UEX, IC3 CH340C, J1 USB-C_DONLY918-418K2022Y40000, Q1 MMDT3904, Q6 DMG2305UX, U1 ESP-12S

Commit message: new
Parts:
- removed D1: 1N5819WS, diode:SOD323-R
- removed SLEEP: JUMPER-SMT_2_NO_NO-SILK, LasKKit-Connectors:SMT-JUMPER_2_NO_NO-SILK
- removed U1: ESP-12S, LasKKit-Modules:ESP12-SMD
- added C6: 100nF, rcl:C0603
- added C7: 47uF, rcl:C0603
- added ESP32: ESP32-WROOM-32D, LasKKit-Modules:ESP32WROOM32D
- added Q2, Q3, Q4, Q5: AO3404A, SparkFun-DiscreteSemi:SOT23-3
- added R10, R7: 100k, rcl:R0402
- added R6: 10k, rcl:R0402
- added U$1: (no value), LasKKit-Aesthetics:LASKKIT_20MM_SILKSCREEN
- added U$2: (no value), LasKKit-Aesthetics:LASKAKIT_HEART_4MM
- C1: value 100nF -> 20p; device rcl:C0603 -> rcl:C0402
- C2: value 10uF -> 20p; device rcl:C0603 -> rcl:C0402
- I2C: value JST-XH-4 -> JST-PH-4; device LasKKit-Connectors:B4B-XH-A -> LasKKit-Connectors:B4B-PH-K
- Q6: value DMG2305UX -> 12MHz; device transistor-power:SUPER-SOT3 -> crystal-geyer_V1_0:3.2X2.5_KX-7
- R3: value 4k7 -> 100k
- R5: value 2k7 -> 10k
- R8: value 470 -> 100k
- moved C1 40.5 mm to (2.67, 5.82), turned to 180 degrees
- moved Q6 37.0 mm to (2.64, 8.20), turned to 180 degrees
- moved C2 35.6 mm to (3.86, 10.6), turned to 180 degrees
- moved C10 30.9 mm to (3.86, 64.9), turned to 270 degrees
- moved IC1 28.4 mm to (6.63, 62.0), turned to 0 degrees
- moved R12 27.8 mm to (-14.3, 41.1)
- moved R13 27.6 mm to (-15.6, 41.1)
- moved RESET 24.0 mm to (12.2, 70.2), turned to 270 degrees
- moved R5 21.4 mm to (-4.27, 46.6), turned to 270 degrees
- moved C9 21.4 mm to (3.84, 59.1), turned to 90 degrees
- moved R4 21.3 mm to (-7.67, 46.6)
- moved R3 21.2 mm to (1.85, 46.6), turned to 90 degrees
- moved C3 11.7 mm to (7.19, 18.3)
- moved LDO 11.7 mm to (7.21, 22.7)
- moved C4 11.7 mm to (7.21, 26.1)
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Connections:
- removed net ADC: U1.ADC
- removed net CH_PD: R2.2, U1.CH_PD
- removed net GPIO0: Q1.3, R4.2, U1.GPIO0
- removed net GPIO12: U1.GPIO12, YELLOW1.A, YELLOW2.A
- removed net GPIO13: RED1.A, RED2.A, U1.GPIO13
- removed net GPIO14: GREEN1.A, GREEN2.A, U1.GPIO14
- removed net GPIO15: R5.1, U1.GPIO15
- removed net GPIO16: R8.2, U1.GPIO16
- removed net GPIO2: Q6.1, R3.2, U1.GPIO2
- removed net GPIO4: I2C.4, R12.1, U1.GPIO4
- removed net GPIO5: I2C.3, R13.1, U1.GPIO5
- removed net RST: C5.2, Q1.6, R1.2, RESET.2, SLEEP.1, U1.RESET
- removed net RX: IC1.7, R18.1, U1.RXD0
- removed net TX: IC1.6, R19.1, U1.TXD0
- new net EN: C5.2, ESP32.3, Q1.6, R1.2, RESET.2
- new net IO0: ESP32.25, Q1.3
- new net IO12: ESP32.14, R2.2
- new net IO13: ESP32.16
- new net IO14: ESP32.13
- new net IO15: ESP32.23
- new net IO16: ESP32.27, IC1.7
- new net IO17: ESP32.28, IC1.6
- new net IO18: ESP32.30
- new net IO19: ESP32.31
- new net IO2: ESP32.24
- new net IO21: ESP32.33, I2C.1, R12.1
- new net IO22: ESP32.36, I2C.2, R13.1
- new net IO23: ESP32.37
- new net IO25: ESP32.10, R4.1
- new net IO26: ESP32.11, R5.1
- new net IO27: ESP32.12, R6.1
- new net IO32: ESP32.8
- new net IO33: ESP32.9
- new net IO34: ESP32.6
- new net IO35: ESP32.7
- new net IO4: ESP32.26
- new net IO5: ESP32.29
- new net N$10: Q4.1, R5.2, R8.2
- new net N$17: Q3.1, R4.2, R7.2
- new net N$2: D3.A, FAN.2, Q2.3
- new net N$3: Q2.1, R2.1, R3.1
- new net N$4: C1.2, IC3.7, Q6.3
- new net N$5: Q5.3, R15.2, R22.2
- new net N$7: Q3.3, R17.2, R20.2
- new net N$9: Q5.1, R10.2, R6.2
- new net RXD0: ESP32.34, R18.1
- new net SENSOR_VN: ESP32.5
- new net SENSOR_VP: ESP32.4
- new net TXD0: ESP32.35, R19.1
- net +3V3: now also C6.1, C7.1, ESP32.2, GREEN1.A, GREEN2.A, I2C.3, RED1.A, RED2.A, YELLOW1.A, YELLOW2.A; no longer C1.1, C2.1, I2C.2, R2.1, R3.1, R4.1, U1.VCC
- net +5V: now also D3.C, FAN.1; no longer D1.C, Q6.2
- net GND: now also C1.1, C2.1, C6.2, C7.2, ESP32.1, ESP32.15, ESP32.38, ESP32.39, I2C.4, Q2.2, Q3.2, Q4.2, Q5.2, R10.1, R3.2, R7.1, R8.1; no longer C1.2, C2.2, D3.A, FAN.2, I2C.1, R15.2, R16.1, R17.2, R20.2, R21.1, R22.2, R5.2, U1.GND
- net N$18: now also C2.2, IC3.8, Q6.1; no longer D1.A, D3.C, FAN.1, Q6.3
- net N$6: now also Q4.3, R16.1, R21.1; no longer R8.1, SLEEP.2
- net RX_: now also SENSOR.2; no longer SENSOR.1
- net TX_: now also SENSOR.1; no longer SENSOR.2
Routing:
- net EN: track 0.00 -> 75.3 mm, vias 0 -> 2
- net TX: track 65.6 -> 0.00 mm, vias 2 -> 0
- net RX: track 63.6 -> 0.00 mm, vias 2 -> 0
- net RST: track 59.7 -> 0.00 mm
- net IO0: track 0.00 -> 54.3 mm, vias 0 -> 2
- net RXD0: track 0.00 -> 52.8 mm, vias 0 -> 2
- net GPIO0: track 51.8 -> 0.00 mm, vias 2 -> 0
- net TXD0: track 0.00 -> 50.9 mm, vias 0 -> 2
- net +5V: track 146.8 -> 105.7 mm, vias 6 -> 2
- net GPIO2: track 41.0 -> 0.00 mm, vias 2 -> 0
- net IO22: track 0.00 -> 38.7 mm, vias 0 -> 1
- net IO21: track 0.00 -> 33.5 mm, vias 0 -> 1
- net GPIO4: track 32.3 -> 0.00 mm, vias 1 -> 0
- net GPIO5: track 30.7 -> 0.00 mm, vias 1 -> 0
- net TX_: track 37.5 -> 7.89 mm, vias 2 -> 0
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Other:
- board size 30 x 75.6 mm -> 33 x 75.6 mm

Commit message: first working
Parts:
- R12, R13, R15, R16, R17, R20, R21, R22: device rcl:R0402 -> rcl:R0603
- R18, R19: device rcl:R0603 -> rcl:R0402
- moved I2C 34.6 mm to (-13.0, 69.5), turned to 180 degrees
- moved R12 26.2 mm to (-10.0, 67.0), flipped to the bottom, turned to 270 degrees
- moved R13 26.1 mm to (-12.0, 67.0), flipped to the bottom, turned to 270 degrees
- moved SENSOR 16.4 mm to (9.53, 68.7), turned to 0 degrees
- moved RESET 13.0 mm to (-0.51, 72.6), turned to 0 degrees
- moved D3 12.7 mm to (7.01, 53.9)
- moved FAN 12.7 mm to (9.39, 53.9)
- moved C6 4.90 mm to (-13.2, 42.0), turned to 0 degrees
- moved C9 2.49 mm to (3.84, 56.6)
- moved ESP32 2.06 mm to (-10.7, 57.0)
- moved C5 2.05 mm to (-11.4, 46.4)
- moved R1 2.05 mm to (-13.9, 46.4)
- moved C7 1.80 mm to (-13.2, 44.0)
- moved Q3 1.80 mm to (-8.61, 41.8)
- moved Q4 1.80 mm to (-5.21, 41.8)
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Connections:
- net IO16 renamed RX2
- net IO17 renamed TX2
- net N$5 renamed R
- net N$6 renamed Y
- net N$7 renamed G
- removed net RX_: IC1.2, SENSOR.2
- removed net TX_: IC1.3, SENSOR.1
- new net RX: IC1.3, SENSOR.2
- new net TX: IC1.2, SENSOR.1
- net +3V3: now also I2C.2; no longer I2C.3
- net GND: now also I2C.1; no longer I2C.4
- net IO21: now also I2C.4; no longer I2C.1
- net IO22: now also I2C.3; no longer I2C.2
Routing:
- net IO22: track 38.7 -> 6.36 mm, vias 1 -> 0
- net IO21: track 33.5 -> 5.97 mm, vias 1 -> 0
- net +3V3: track 150.7 -> 172.9 mm, vias 3 -> 4
- net RX: track 0.00 -> 11.0 mm
- net EN: track 75.3 -> 64.4 mm
- net TX: track 0.00 -> 10.7 mm
- net RX_: track 9.84 -> 0.00 mm
- net +5V: track 105.7 -> 115.4 mm
- net N$2: track 9.08 -> 17.9 mm
- net TX_: track 7.89 -> 0.00 mm
- net TX2: track 17.9 -> 15.7 mm
- net RX2: track 15.3 -> 13.5 mm
- net Y: track 12.8 -> 14.3 mm
- net IO25: track 4.17 -> 5.21 mm
- net IO12: track 5.54 -> 4.54 mm
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Other:
- outline, holes or cut-outs redrawn
- board text removed: "3V3"
- board text removed: "GND"
- board text removed: "SCL"
- board text removed: "SDA"

Commit message: connectors pos
Parts:
- I2C: value JST-PH-4 -> (none); device LasKKit-Connectors:B4B-PH-K -> LasKKit-Connectors:1X04
- moved C6 2.06 mm to (-13.3, 44.0)
- moved C7 2.06 mm to (-13.3, 42.0)
- moved R12 1.00 mm to (-9.14, 66.5)
- moved I2C 0.49 mm to (-12.7, 69.2)
- moved R13 0.46 mm to (-12.1, 66.5)
Connections:
- net +3V3: now also I2C.4; no longer I2C.2
- net GND: now also I2C.3; no longer I2C.1
- net IO21: now also I2C.1; no longer I2C.4
- net IO22: now also I2C.2; no longer I2C.3
Routing:
- net +3V3: track 172.9 -> 174.5 mm

Commit message: updaterd
Routing:
- net GND: track 25.0 -> 25.5 mm
Other:
- board size 33 x 75.6 mm -> 33 x 74.9 mm
Changed lines of the file:
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@@
 <board>
 <plain>
-<wire x1="-6.75" y1="-1" x2="6.75" y2="-1" width="0" layer="20"/>
-<wire x1="6.75" y1="-1" x2="6.75" y2="2.25" width="0" layer="20"/>
-<wire x1="-6.75" y1="2.25" x2="-6.75" y2="-1" width="0" layer="20"/>
+<wire x1="-6.75" y1="-0.3" x2="6.75" y2="-0.3" width="0" layer="20"/>
+<wire x1="6.75" y1="-0.3" x2="6.75" y2="2.25" width="0" layer="20"/>
+<wire x1="-6.75" y1="2.25" x2="-6.75" y2="-0.3" width="0" layer="20"/>
 <wire x1="-7.75" y1="3.25" x2="-10" y2="3.25" width="0" layer="20"/>
 <wire x1="7.75" y1="3.25" x2="10" y2="3.25" width="0" layer="20"/>
@@
 </element>
 <element name="ESP32" library="LasKKit-Modules" library_urn="urn:adsk.eagle:library:21721098" package="ESP32WROOM32D" package3d_urn="urn:adsk.eagle:package:28305005/6" value="ESP32-WROOM-32D" x="-10.684" y="56.9722" smashed="yes">
-<attribute name="ARROW_PART_NUMBER" value="" x="-10.684" y="52.07" size="1.778" layer="27" display="off"/>
-<attribute name="ARROW_PRICE-STOCK" value="" x="-10.684" y="52.07" size="1.778" layer="27" display="off"/>
-<attribute name="DESCRIPTION" value="WiFi Modules (802.11) SMD Module, ESP32-D0WD, 32Mbits SPI flash, UART mode, PCB antenna" x="-10.684" y="52.07" size="1.778" layer="27" display="off"/>
-<attribute name="HEIGHT" value="3.1mm" x="-10.684" y="52.07" size="1.778" layer="27" display="off"/>
 <attribute name="LCSC_PART" value="C82899" x="-10.684" y="52.07" size="1.778" layer="27" display="off"/>
-<attribute name="MANUFACTURER_NAME" value="Espressif Systems" x="-10.684" y="52.07" size="1.778" layer="27" display="off"/>
-<attribute name="MANUFACTURER_PART_NUMBER" value="ESP32-WROOM-32D" x="-10.684" y="52.07" size="1.778" layer="27" display="off"/>
-<attribute name="MOUSER_PART_NUMBER" value="N/A" x="-10.684" y="52.07" size="1.778" layer="27" display="off"/>
-<attribute name="MOUSER_PRICE-STOCK" value="https://www.mouser.co.uk/ProductDetail/Espressif-Systems/ESP32-WROOM-32D?qs=MLItCLRbWszx2KabkKPu5A%3D%3D" x="-10.684" y="52.07" size="1.778" layer="27" display="off"/>
 <attribute name="NAME" x="3.5064" y="49.5134" size="0.8128" layer="25" font="vector" ratio="15" rot="R90" align="center"/>
 <attribute name="VALUE" x="-19.484" y="56.6722" size="1.27" layer="27" rot="R90" align="center"/>
@@
 <wire x1="2" y1="3.53" x2="3.5052" y2="3.53" width="0.254" layer="1"/>
 <wire x1="3.5052" y1="3.53" x2="3.5052" y2="3.556" width="0.254" layer="1"/>
-<wire x1="2" y1="-0.33" x2="3.4036" y2="-0.33" width="0.254" layer="1"/>
-<wire x1="3.4036" y1="-0.33" x2="3.4036" y2="-0.3302" width="0.254" layer="1"/>
-<wire x1="-2" y1="-0.33" x2="-3.429" y2="-0.33" width="0.254" layer="1"/>
-<wire x1="-3.429" y1="-0.33" x2="-3.429" y2="-0.3302" width="0.254" layer="1"/>
-<wire x1="-2" y1="-0.33" x2="-3.3782" y2="-0.33" width="0.254" layer="16"/>
-<wire x1="2" y1="-0.33" x2="3.4798" y2="-0.33" width="0.254" layer="16"/>
-<wire x1="3.4798" y1="-0.33" x2="3.4798" y2="-0.3302" width="0.254" layer="16"/>
 <wire x1="2" y1="3.53" x2="2" y2="4.445" width="0.254" layer="16"/>
 <wire x1="2" y1="4.445" x2="1.9812" y2="4.445" width="0.254" layer="16"/>
@@
 <via x="-1.4732" y="37.6174" extent="1-16" drill="0.3"/>
 <contactref element="I2C" pad="3"/>
+<wire x1="-2" y1="-0.33" x2="-2.4316" y2="0.1016" width="0.254" layer="1"/>
+<wire x1="-2.4316" y1="0.1016" x2="-3.4036" y2="0.1016" width="0.254" layer="1"/>
+<wire x1="2" y1="-0.33" x2="2.4316" y2="0.1016" width="0.254" layer="1"/>
+<wire x1="2.4316" y1="0.1016" x2="3.3528" y2="0.1016" width="0.254" layer="1"/>
+<wire x1="2" y1="-0.33" x2="2.4316" y2="0.1016" width="0.254" layer="16"/>
+<wire x1="2.4316" y1="0.1016" x2="3.3782" y2="0.1016" width="0.254" layer="16"/>
+<wire x1="-2" y1="-0.33" x2="-2.4316" y2="0.1016" width="0.254" layer="16"/>
+<wire x1="-2.4316" y1="0.1016" x2="-3.3782" y2="0.1016" width="0.254" layer="16"/>
 </signal>
 <signal name="+3V3">
